Commit message: Refactor navigation parameters and update URDF for improved vehicle dynamics and mapping

File: resource/tesla_webots.urdf (robot description, URDF)
Before this commit: robot Tesla Webots, 3 links, 2 joints
Joints:
- joint lidar_front_joint: origin xyz=-0.1 0 0.1 rpy=0 0 0 -> xyz=2.05 0 0.1 rpy=0 0 0
- joint lidar_rear_joint: origin xyz=-4.73 0 0.1 rpy=0 0 3.14159 -> xyz=-2.58 0 0.1 rpy=0 0 3.14159

Commit message: Refactor code structure for improved readability and maintainability

File: resource/tesla_webots.urdf (robot description, URDF)
Before this commit: robot Tesla Webots, 3 links, 2 joints
Links:
- added link gps_link
- added link imu_link
Joints:
- added joint gps_joint: type fixed, parent base_link, child gps_link, origin xyz=-0.35 0 0.95 rpy=0 0 0
- added joint imu_joint: type fixed, parent base_link, child imu_link, origin xyz=-0.35 0 0.95 rpy=0 0 0
